File: LR4HP.sch (KiCad schematic (older format))
At the start: 13 parts, among them U9 NE5532

Commit message: Board is placed and about half-routed
Connections:
- net FB1: now reaches C47.2, R41.1, U9.1, U9.2 (-)
- net VP1: now reaches C50.1, R44.1, U9.3 (+)
- net VP2: now reaches C48.1, R43.1, U9.5 (+)
Changed lines of the file:
@@
 AR Path="/61597701/61581F20" Ref="U10"  Part="3"
 AR Path="/615C4B54/61581F20" Ref="U?"  Part="3"
-F 0 "U9" H 3358 4996 50  0000 L CNN
+F 0 "U10" H 3358 4996 50  0000 L CNN
 F 1 "NE5532" H 3358 4905 50  0000 L CNN
 F 2 "Housings_DIP:DIP-8_W7.62mm_Socket" H 3400 4950 50  0001 C CNN
@@
 AR Path="/61597701/615A630E" Ref="C58"  Part="1"
 AR Path="/615C4B54/615A630E" Ref="C?"  Part="1"
-F 0 "C52" H 2865 5246 50  0000 L CNN
+F 0 "C58" H 2865 5246 50  0000 L CNN
 F 1 "100n" H 2865 5155 50  0000 L CNN
 F 2 "Capacitors_SMD:C_0805" H 2788 5050 50  0001 C CNN
@@
 AR Path="/61597701/61593BE2" Ref="R51"  Part="1"
 AR Path="/615C4B54/61593BE2" Ref="R?"  Part="1"
-F 0 "R45" H 4070 2946 50  0000 L CNN
+F 0 "R51" H 4070 2946 50  0000 L CNN
 F 1 "R" H 4070 2855 50  0000 L CNN
 F 2 "Resistors_SMD:R_0805" V 3930 2900 50  0001 C CNN
@@
 AR Path="/61597701/615935AE" Ref="R50"  Part="1"
 AR Path="/615C4B54/615935AE" Ref="R?"  Part="1"
-F 0 "R44" H 4070 2546 50  0000 L CNN
+F 0 "R50" H 4070 2546 50  0000 L CNN
 F 1 "R" H 4070 2455 50  0000 L CNN
 F 2 "Resistors_SMD:R_0805" V 3930 2500 50  0001 C CNN
@@
 AR Path="/61597701/61592F52" Ref="R47"  Part="1"
 AR Path="/615C4B54/61592F52" Ref="R?"  Part="1"
-F 0 "R41" H 3470 1896 50  0000 L CNN
+F 0 "R47" H 3470 1896 50  0000 L CNN
 F 1 "R" H 3470 1805 50  0000 L CNN
 F 2 "Resistors_SMD:R_0805" V 3330 1850 50  0001 C CNN
@@
 AR Path="/61597701/61590C79" Ref="C56"  Part="1"
 AR Path="/615C4B54/61590C79" Ref="C?"  Part="1"
-F 0 "C50" V 3398 2200 50  0000 C CNN
+F 0 "C56" V 3398 2200 50  0000 C CNN
 F 1 "C" V 3489 2200 50  0000 C CNN
 F 2 "Capacitors_SMD:C_1210_HandSoldering" H 3688 2050 50  0001 C CNN
@@
 AR Path="/61597701/6158BBA5" Ref="C55"  Part="1"
 AR Path="/615C4B54/6158BBA5" Ref="C?"  Part="1"
-F 0 "C49" V 2848 2200 50  0000 C CNN
+F 0 "C55" V 2848 2200 50  0000 C CNN
 F 1 "C" V 2939 2200 50  0000 C CNN
 F 2 "Capacitors_SMD:C_1210_HandSoldering" H 3138 2050 50  0001 C CNN
@@
 AR Path="/61597701/61581F14" Ref="U10"  Part="1"
 AR Path="/615C4B54/61581F14" Ref="U?"  Part="1"
-F 0 "U9" H 4600 1733 50  0000 C CNN
+F 0 "U10" H 4600 1733 50  0000 C CNN
 F 1 "NE5532" H 4600 1824 50  0000 C CNN
 F 2 "Housings_DIP:DIP-8_W7.62mm_Socket" H 4600 2100 50  0001 C CNN
@@
 AR Path="/61597701/615B29CF" Ref="C54"  Part="1"
 AR Path="/615C4B54/615B29CF" Ref="C?"  Part="1"
-F 0 "C48" V 6548 2150 50  0000 C CNN
+F 0 "C54" V 6548 2150 50  0000 C CNN
 F 1 "C" V 6639 2150 50  0000 C CNN
 F 2 "Capacitors_SMD:C_1210_HandSoldering" H 6838 2000 50  0001 C CNN
@@
 AR Path="/61597701/615B9BE0" Ref="C53"  Part="1"
 AR Path="/615C4B54/615B9BE0" Ref="C?"  Part="1"
-F 0 "C47" V 6048 2150 50  0000 C CNN
+F 0 "C53" V 6048 2150 50  0000 C CNN
 F 1 "C" V 6139 2150 50  0000 C CNN
 F 2 "Capacitors_SMD:C_1210_HandSoldering" H 6338 2000 50  0001 C CNN
@@
 AR Path="/61597701/615C3593" Ref="R48"  Part="1"
 AR Path="/615C4B54/615C3593" Ref="R?"  Part="1"
-F 0 "R42" H 6620 1896 50  0000 L CNN
+F 0 "R48" H 6620 1896 50  0000 L CNN
 F 1 "R" H 6620 1805 50  0000 L CNN
 F 2 "Resistors_SMD:R_0805" V 6480 1850 50  0001 C CNN
@@
 AR Path="/61597701/615C391A" Ref="R49"  Part="1"
 AR Path="/615C4B54/615C391A" Ref="R?"  Part="1"
-F 0 "R43" H 7220 2496 50  0000 L CNN
+F 0 "R49" H 7220 2496 50  0000 L CNN
 F 1 "R" H 7220 2405 50  0000 L CNN
 F 2 "Resistors_SMD:R_0805" V 7080 2450 50  0001 C CNN
@@
 AR Path="/61597701/615C3D1F" Ref="R52"  Part="1"
 AR Path="/615C4B54/615C3D1F" Ref="R?"  Part="1"
-F 0 "R46" H 7220 2946 50  0000 L CNN
+F 0 "R52" H 7220 2946 50  0000 L CNN
 F 1 "R" H 7220 2855 50  0000 L CNN
 F 2 "Resistors_SMD:R_0805" V 7080 2900 50  0001 C CNN
@@
 AR Path="/61597701/615CA1F0" Ref="C57"  Part="1"
 AR Path="/615C4B54/615CA1F0" Ref="C?"  Part="1"
-F 0 "C51" H 2865 4746 50  0000 L CNN
+F 0 "C57" H 2865 4746 50  0000 L CNN
 F 1 "100n" H 2865 4655 50  0000 L CNN
 F 2 "Capacitors_SMD:C_0805" H 2788 4550 50  0001 C CNN
@@
 AR Path="/61597701/61581F1A" Ref="U10"  Part="2"
 AR Path="/615C4B54/61581F1A" Ref="U?"  Part="2"
-F 0 "U9" H 7600 1683 50  0000 C CNN
+F 0 "U10" H 7600 1683 50  0000 C CNN
 F 1 "NE5532" H 7600 1774 50  0000 C CNN
 F 2 "Housings_DIP:DIP-8_W7.62mm_Socket" H 7600 2050 50  0001 C CNN
@@
 Wire Wire Line
 	2450 2200 2950 2200
-Text Notes 5250 3900 0    50   ~ 0
+Text Notes 5200 2700 0    50   ~ 0
 f=1/(pi*2^1.5*R*C)
+Text Label 2650 2200 0    50   ~ 0
+IN
+Text Label 3750 1650 0    50   ~ 0
+FB1
+Text Label 3850 2200 0    50   ~ 0
+VP1
+Text Label 7050 2150 0    50   ~ 0
+VP2
+Text Label 6850 1650 0    50   ~ 0
+FB2
 $EndSCHEMATC
